File: Light Controller/Traffic Light Controller.kicad_pcb (KiCad board)
At the start: 2 copper layers, 107.5 x 82.5 mm, 65 parts, among them J1 Conn_02x08_Odd_Even, J2 Conn_02x08_Odd_Even, J3 Conn_02x05_Odd_Even, J4 +5V, SW1 RST, SW2 OVR, SW3 EN, U1 SM420561N, U2 SM420561N, U3 LM1117DT-3.3

Commit message: Updated 04/21/26 (20:16)
Parts:
- added G***: LOGO, my_footprints:pepe_logo, F.Cu at (212.0, 113.5)
Routing:
- added copper zone on F.Cu, net (none)
Other:
- board text added: "FELIXANDER B. DOLOSO SETH ANDREI V. GEDALANGA 21 April 2026 Computer Engineerig Technology Department Technological University of the Philippines Visayas"
