File: Light Controller Ver9.0/Traffic Light Controller/Traffic Light Controller.kicad_pcb (KiCad board)
At the start: 2 copper layers, 107.5 x 82.5 mm, 65 parts, among them J1 Conn_02x08_Odd_Even, J2 Conn_02x08_Odd_Even, J3 Conn_02x05_Odd_Even, J4 +5V, SW1 RST, SW2 OVR, SW3 EN, U1 SM420561N, U2 SM420561N, U3 LM1117DT-3.3

Commit message: Updated 05/04/26 (16:06)
Routing:
- added copper zone on F.Cu, net /+3.3V
- added copper zone on B.Cu, net GND
- removed copper zone on F.Cu, net (none)
Other:
- board text added: "0.1270 mm / 0.1270 mm"
- board text added: "0.3000 mm"
- board text added: "1.6000 mm"
- board text added: "107.5000 mm x 82.5000 mm"
- board text added: "BOARD CHARACTERISTICS"
- board text added: "Board Thickness:"
- board text added: "Board overall dimensions:"
- board text added: "Castellated pads:"
- board text added: "Copper Finish:"
- board text added: "Copper Layer Count:"
- board text added: "Edge card connectors:"
- board text added: "HAL SnPb"
- board text added: "Impedance Control:"
- board text added: "Min hole diameter:"
- board text added: "Min track/spacing:"
- board text added: "No"
- board text added: "Plated Board Edge:"
